File: hardware/ArcDice.kicad_pcb (KiCad board)
At the start: 2 copper layers, 70 x 70 mm, 26 parts, among them SW1 SW_SPDT, SW2 SW_Push, U1 ATtiny13A-P, U2 TP4056_Module

Commit message: Update hardware design
Routing:
- net /BTN_ROLL: track 15.1 -> 20.4 mm
Changed lines of the file:
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@@
 			(at 0 3.15 0)
 			(layer "F.Fab")
+			(hide yes)
 			(effects
 				(font
@@
 			(at 0 3.15 0)
 			(layer "F.Fab")
+			(hide yes)
 			(effects
 				(font
@@
 			(at 0 3.15 0)
 			(layer "F.Fab")
+			(hide yes)
 			(effects
 				(font
@@
 			(at 0 3.15 0)
 			(layer "F.Fab")
+			(hide yes)
 			(effects
 				(font
@@
 	)
 	(segment
-		(start 126.5 48)
-		(end 121.23 53.27)
+		(start 121.23 53.27)
+		(end 120.06 53.27)
 		(width 0.25)
 		(layer "B.Cu")
@@
 	)
 	(segment
-		(start 121.23 53.27)
-		(end 120.06 53.27)
+		(start 131.75 48)
+		(end 126.5 48)
 		(width 0.25)
 		(layer "B.Cu")
@@
 	)
 	(segment
-		(start 133 48)
-		(end 126.5 48)
+		(start 126.5 48)
+		(end 121.23 53.27)
+		(width 0.25)
+		(layer "B.Cu")
+		(net "/BTN_ROLL")
+	)
+	(segment
+		(start 138.25 48)
+		(end 131.75 48)
 		(width 0.25)
 		(layer "B.Cu")
@@
 	)
 	(segment
+		(start 155.25 66.16)
+		(end 155.25 52.25)
+		(width 0.6)
+		(layer "B.Cu")
+		(net "/SW IN")
+	)
+	(segment
+		(start 166.595 77.505)
+		(end 155.25 66.16)
+		(width 0.6)
+		(layer "B.Cu")
+		(net "/SW IN")
+	)
+	(segment
 		(start 130.25 65.19)
 		(end 130.19 65.19)
@@
 		(net "/BAT_MINUS")
 	)
-	(segment
-		(start 155.25 66.16)
-		(end 155.25 52.25)
-		(width 0.6)
-		(layer "B.Cu")
-		(net "/SW IN")
-	)
-	(segment
-		(start 166.595 77.505)
-		(end 155.25 66.16)
-		(width 0.6)
-		(layer "B.Cu")
-		(net "/SW IN")
-	)
 	(zone

Commit message: logo added
Other:
- board text added: "v2.0"
