File: hardware/ArcDice.kicad_pcb (KiCad board)
At the start: 2 copper layers, 70 x 70 mm, 26 parts, among them SW1 SW_SPDT, SW2 SW_Push, U1 ATtiny13A-P, U2 TP4056_Module

Commit message: hardware: update KiCad schematic, PCB, and project files
Parts:
- H1, H2, H3, H4: footprint MountingHole:MountingHole_2.2mm_M2 -> MountingHole:MountingHole_3.2mm_M3
- moved H1 1.41 mm to (166.0, 44.0)
- moved H2 1.41 mm to (104.0, 106.0)
- moved H3 1.41 mm to (104.0, 44.0)
- moved H4 1.41 mm to (166.0, 106.0)
Other:
- board text added: "ON"

Commit message: hardware: minor PCB update
Other:
- board text added: "PCB ver. v2.1"
- board text removed: "v2.0"
Changed lines of the file:
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@@
 		(layer "Edge.Cuts")
 	)
-	(gr_text "v2.0"
-		(at 157.75 107.75 0)
+	(gr_text "PCB ver. v2.1"
+		(at 151.5 107.75 0)
 		(layer "F.SilkS")
 		(effects
